Commit message: limits done, collisions semi-done, issues

File: urdf/stick.urdf (robot description, URDF)
Before this commit: robot my_kuka_robot, 9 links, 8 joints
Joints:
- joint link1_to_link2: limit (none) -> lower=-1.57 upper=1.57 effort=0.0 velocity=0.0; type continuous -> revolute
- joint link3_to_link4: limit (none) -> lower=-1.57 upper=1.57 effort=0.0 velocity=0.0; type continuous -> revolute
- joint link5_to_link6: limit (none) -> lower=-1.57 upper=1.57 effort=0.0 velocity=0.0; type continuous -> revolute

Commit message: updated collisions

File: urdf/stick.urdf (robot description, URDF)
Before this commit: robot my_kuka_robot, 9 links, 8 joints
Links:
- link base_link: geometry collision mesh filename=package://kuka_stick_description/meshes/simplified/simplifi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 scale=1.0 1.0 1.0; visual mesh filename=package://kuka_stick_description/meshes/link_0.dae scale=1.0 1.0 1.0
- link link_1: geometry collision mesh filename=package://kuka_stick_description/meshes/simplified/simplifi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 scale=1.0 1.0 1.0; visual mesh filename=package://kuka_stick_description/meshes/link_1.dae scale=1.0 1.0 1.0
- link link_2: geometry collision mesh filename=package://kuka_stick_description/meshes/simplified/simplifi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 scale=1.0 1.0 1.0; visual mesh filename=package://kuka_stick_description/meshes/link_2.dae scale=1.0 1.0 1.0
- link link_3: geometry collision mesh filename=package://kuka_stick_description/meshes/simplified/simplifi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 scale=1.0 1.0 1.0; visual mesh filename=package://kuka_stick_description/meshes/link_3.dae scale=1.0 1.0 1.0
- link link_4: geometry collision mesh filename=package://kuka_stick_description/meshes/simplified/simplifi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 scale=1.0 1.0 1.0; visual mesh filename=package://kuka_stick_description/meshes/link_4.dae scale=1.0 1.0 1.0
- link link_5: geometry collision mesh filename=package://kuka_stick_description/meshes/simplified/simplifi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 scale=1.0 1.0 1.0; visual mesh filename=package://kuka_stick_description/meshes/link_5.dae scale=1.0 1.0 1.0
- link link_6: geometry collision mesh filename=package://kuka_stick_description/meshes/simplified/simplifi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 scale=1.0 1.0 1.0; visual mesh filename=package://kuka_stick_description/meshes/link_6.dae scale=1.0 1.0 1.0
- link link_7: geometry collision mesh filename=package://kuka_stick_description/meshes/simplified/simplifi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 scale=1.0 1.0 1.0; visual mesh filename=package://kuka_stick_description/meshes/link_7.dae scale=1.0 1.0 1.0
